File: Eagle/WiringDiagram.sch (EAGLE design)
At the start: 10 parts

Commit message: Eagle - More work on wiring diagram
Parts:
- added U$4: MAX3232, parts:MAX3232
- renumbered U$2 to LEFT_ESC, U$3 to RIGHT_ESC
Connections:
- new net LEFT_PWM: LEFT_ESC.PWM, U$1.OUT1
- new net N$10: U$4.DE9-8, U$5.CTS
- new net N$11: U$1.RX1-I, U$6.D1/TX
- new net N$12: U$4.RX, U$6.D2
- new net N$13: U$4.TX, U$6.D3
- new net N$14: U$1.TX1-O, U$6.D0/RX
- new net N$15: RIGHT_ESC.DIR
- new net N$18: LEFT_ESC.DIR
- new net N$5: U$4.DE9-1, U$5.DCD
- new net N$6: U$4.DE9-2, U$5.TXD
- new net N$7: U$4.DE9-3, U$5.RXD
- new net N$8: U$4.DE9-4, U$5.DTR
- new net N$9: U$4.DE9-7, U$5.RTS
- new net RIGHT_PWM: RIGHT_ESC.PWM, U$1.OUT3
- net 5V: now also U$1.JP_VCC@1, U$1.JP_VCC@2, U$4.VCC, U$5.VCC
- net GND: now also LEFT_ESC.GND, RIGHT_ESC.GND, U$1.GND@5, U$1.GND@6, U$4.GND, U$5.GND, U$6.GND@1, U$6.GND@2; no longer U$6.GND, U$6.GND2

Commit message: Misc
Parts:
- removed LEFT_ESC, RIGHT_ESC: BESC30-R1, parts:BESC30-R1
- removed U$6: XTWDUINO_NANO_3, parts:XTWDUINO_NANO_3
- added U$2: SOLARPANEL, parts:SOLARPANEL
- added U$3, U$7: BESC30-R1, parts:BESC30-R1
Connections:
- removed net 5V: PSU.5V_B_POS, U$1.JP_VCC@1, U$1.JP_VCC@2, U$4.VCC, U$5.VCC, U$6.VIN
- removed net GND: LEFT_ESC.GND, PSU.5V_B_NEG, RIGHT_ESC.GND, U$1.GND@5, U$1.GND@6, U$4.GND, U$5.GND, U$6.GND@1, U$6.GND@2
- removed net LEFT_PWM: LEFT_ESC.PWM, U$1.OUT1
- removed net N$18: LEFT_ESC.DIR
- removed net RIGHT_PWM: RIGHT_ESC.PWM, U$1.OUT3
- new net 5V_A: PSU.5V_A_POS, U$5.VCC
- new net 5V_B: PSU.5V_B_POS, U$1.JP_VCC@1, U$1.JP_VCC@2
- new net ESC_LEFT0: U$1.GND_OUT, U$3.GND
- new net ESC_LEFT1: U$1.OUT1, U$3.PWM
- new net ESC_LEFT2: U$1.VCC_OUT, U$3.5V_BEC
- new net ESC_RIGHT0: U$7.5V_BEC, U$7.GND
- new net ESC_RIGHT1: U$1.OUT3, U$7.PWM
- new net GND_A: PSU.5V_A_NEG, U$5.GND
- new net GPS0: U$1.P$63, U$1.P$64
- new net GPS2: U$1.P$62
- new net GPS3: U$1.P$61
- new net GPS4: U$1.P$60
- new net N$16: U$2.POS
- new net N$17: PSU.PANEL_NEG, U$2.NEG
- new net TELEM0: U$1.VCC@1
- new net TELEM1: U$1.TX1-O
- new net TELEM2: U$1.RX1-I
- new net TELEM3: U$1.NC@1
- new net TELEM4: U$1.GND
- net N$11: now also U$4.RX; no longer U$1.RX1-I, U$6.D1/TX
- net N$12: now also U$1.P$52, U$4.GND; no longer U$4.RX, U$6.D2
- net N$13: no longer U$6.D3
- net N$14: now also U$4.VCC; no longer U$1.TX1-O, U$6.D0/RX
- net N$15: now also PSU.5V_B_NEG, U$1.GND@5, U$1.GND@6; no longer RIGHT_ESC.DIR
- net N$3: now also U$3.NEG, U$7.NEG; no longer LEFT_ESC.12V_NEG, RIGHT_ESC.12V_NEG
- net N$4: now also U$3.POS, U$7.POS; no longer LEFT_ESC.12V_POS, RIGHT_ESC.12V_POS
Other:
- note added: "10A max"
- note added: "DC13-4S"
- note added: "DF13-5S"
- note added: "DF13-6S"
- note added: "Hookup"
- note added: "Modem"
- note added: "Motor Controllers (ESC)"
- note added: "NC"
- note added: "Provided"
- note added: "RJ45 -> DE9+DC Cable (provided)"
- note added: "Spade connectors"
- note added: "USB -> DF13-6S"
- note added: "USB -> Plug"
- note added: "USB Socket"
- note added: "~10A max (should never run at that)"

Commit message: Writing dickery
Parts:
- renumbered U$4 to MAX232
Other:
- note added: "BEC (to APM)"
- note added: "Gender Changer+Crossover"
- note added: "USB -> DF13-6S (optional)"
- note removed: "USB -> DF13-6S"
Changed lines of the file:
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@@
 <part name="BATT3" library="parts" deviceset="HT12V3.3" device=""/>
 <part name="BATT4" library="parts" deviceset="HT12V3.3" device=""/>
-<part name="U$4" library="parts" deviceset="MAX3232" device=""/>
+<part name="MAX232" library="parts" deviceset="MAX3232" device=""/>
 <part name="U$2" library="parts" deviceset="SOLARPANEL" device=""/>
 <part name="U$3" library="parts" deviceset="BESC30-R1" device=""/>
@@
 <text x="-17.78" y="-58.42" size="1.778" layer="91">Hookup</text>
 <text x="-5.08" y="-15.24" size="1.778" layer="91">USB -&gt; Plug</text>
-<text x="-22.86" y="10.16" size="1.778" layer="91">USB -&gt; DF13-6S</text>
+<text x="-22.86" y="10.16" size="1.778" layer="91">USB -&gt; DF13-6S
+(optional)</text>
 <text x="-58.42" y="17.78" size="1.778" layer="91">Provided</text>
 <text x="33.02" y="-50.8" size="1.778" layer="91">NC</text>
@@
 <text x="17.78" y="25.4" size="1.778" layer="91">DC13-4S</text>
 <text x="-2.54" y="25.4" size="1.778" layer="91">DF13-6S</text>
+<text x="-50.8" y="58.42" size="1.778" layer="91">BEC (to APM)</text>
+<text x="27.94" y="-68.58" size="1.778" layer="91">Gender Changer+Crossover</text>
 </plain>
 <instances>
@@
 <instance part="BATT3" gate="G$1" x="-127" y="2.54"/>
 <instance part="BATT4" gate="G$1" x="-127" y="-25.4"/>
-<instance part="U$4" gate="G$1" x="12.7" y="-48.26"/>
+<instance part="MAX232" gate="G$1" x="12.7" y="-48.26"/>
 <instance part="U$2" gate="G$1" x="-124.46" y="-58.42" rot="R270"/>
 <instance part="U$3" gate="G$1" x="154.94" y="7.62"/>
@@
 <net name="N$5" class="0">
 <segment>
-<pinref part="U$4" gate="G$1" pin="DE9-1"/>
+<pinref part="MAX232" gate="G$1" pin="DE9-1"/>
 <wire x1="33.02" y1="-40.64" x2="35.56" y2="-40.64" width="0.1524" layer="91"/>
 <wire x1="35.56" y1="-40.64" x2="48.26" y2="-55.88" width="0.1524" layer="91"/>
@@
 <net name="N$6" class="0">
 <segment>
-<pinref part="U$4" gate="G$1" pin="DE9-2"/>
+<pinref part="MAX232" gate="G$1" pin="DE9-2"/>
 <wire x1="33.02" y1="-43.18" x2="43.18" y2="-43.18" width="0.1524" layer="91"/>
 <wire x1="43.18" y1="-43.18" x2="45.72" y2="-45.72" width="0.1524" layer="91"/>
@@
 <net name="N$7" class="0">
 <segment>
-<pinref part="U$4" gate="G$1" pin="DE9-3"/>
+<pinref part="MAX232" gate="G$1" pin="DE9-3"/>
 <wire x1="33.02" y1="-45.72" x2="43.18" y2="-45.72" width="0.1524" layer="91"/>
 <wire x1="43.18" y1="-45.72" x2="45.72" y2="-48.26" width="0.1524" layer="91"/>
@@
 <net name="N$8" class="0">
 <segment>
-<pinref part="U$4" gate="G$1" pin="DE9-4"/>
+<pinref part="MAX232" gate="G$1" pin="DE9-4"/>
 <wire x1="33.02" y1="-48.26" x2="43.18" y2="-48.26" width="0.1524" layer="91"/>
 <pinref part="U$5" gate="G$1" pin="DTR"/>
@@
 <net name="N$9" class="0">
 <segment>
-<pinref part="U$4" gate="G$1" pin="DE9-7"/>
+<pinref part="MAX232" gate="G$1" pin="DE9-7"/>
 <wire x1="33.02" y1="-55.88" x2="38.1" y2="-55.88" width="0.1524" layer="91"/>
 <wire x1="38.1" y1="-55.88" x2="50.8" y2="-43.18" width="0.1524" layer="91"/>
@@
 <net name="N$10" class="0">
 <segment>
-<pinref part="U$4" gate="G$1" pin="DE9-8"/>
+<pinref part="MAX232" gate="G$1" pin="DE9-8"/>
 <wire x1="33.02" y1="-58.42" x2="35.56" y2="-58.42" width="0.1524" layer="91"/>
 <wire x1="35.56" y1="-58.42" x2="35.56" y2="-55.88" width="0.1524" layer="91"/>
@@
 <net name="N$13" class="0">
 <segment>
-<pinref part="U$4" gate="G$1" pin="TX"/>
+<pinref part="MAX232" gate="G$1" pin="TX"/>
 <wire x1="-10.16" y1="-48.26" x2="-12.7" y2="-48.26" width="0.1524" layer="91"/>
 <wire x1="-12.7" y1="-48.26" x2="-12.7" y2="-30.48" width="0.1524" layer="91"/>
@@
 <net name="N$11" class="0">
 <segment>
-<pinref part="U$4" gate="G$1" pin="RX"/>
+<pinref part="MAX232" gate="G$1" pin="RX"/>
 <wire x1="-10.16" y1="-50.8" x2="-15.24" y2="-50.8" width="0.1524" layer="91"/>
 <wire x1="-15.24" y1="-50.8" x2="-15.24" y2="-27.94" width="0.1524" layer="91"/>
@@
 <net name="N$12" class="0">
 <segment>
-<pinref part="U$4" gate="G$1" pin="GND"/>
+<pinref part="MAX232" gate="G$1" pin="GND"/>
 <label x="-12.7" y="-53.34" size="1.778" layer="95"/>
 <wire x1="-10.16" y1="-53.34" x2="-17.78" y2="-53.34" width="0.1524" layer="91"/>
@@
 <net name="N$14" class="0">
 <segment>
-<pinref part="U$4" gate="G$1" pin="VCC"/>
+<pinref part="MAX232" gate="G$1" pin="VCC"/>
 <wire x1="-10.16" y1="-45.72" x2="-10.16" y2="-33.02" width="0.1524" layer="91"/>
 <wire x1="-10.16" y1="-33.02" x2="25.4" y2="-33.02" width="0.1524" layer="91"/>

Commit message: Wiring diragram, meh
Connections:
- removed net 5V_B: PSU.5V_B_POS, U$1.JP_VCC@1, U$1.JP_VCC@2
- removed net N$15 (its old number): PSU.5V_B_NEG, U$1.GND@5, U$1.GND@6
- new net N$18: U$1.JP_VCC@1, U$1.JP_VCC@2
- new net N$19: U$1.GND@5, U$1.GND@6
- net N$11: now also U$1.P$53
- net N$13: now also U$1.P$54
Other:
- note added: "20AWG figure-8"
- note added: "Connector SAE Bullet"
- note added: "Connector: SAE Bullet"
- note added: "Custom: RJ45->DE9 Male + USB"
- note added: "Extended SAE bullet cable length TBD"
- note added: "Hookup wire"
- note added: "Join at PSU"
- note added: "Powered by BEC"
- note added: "To radio board"
- note added: "hull"
- note removed: "Gender Changer+Crossover"
- note removed: "RJ45 -> DE9+DC Cable (provided)"
- note removed: "USB -> DF13-6S (optional)"
